File: eagle_files/beeshield.brd (EAGLE design)
At the start: 32.2 x 41.6 mm, 14 parts

Commit message: new eagle files
Routing:
- net IO2: track 51.3 -> 55.2 mm
- net VCC: track 83.6 -> 87.6 mm
- net GND: track 113.2 -> 116.9 mm
- net IO3: track 49.0 -> 51.4 mm
- net IO0: track 37.4 -> 39.4 mm
- net IO1: track 37.9 -> 39.5 mm
